File: Schematic_motor_driver.brd (EAGLE design)
At the start: 50 x 50 mm, 23 parts, among them Q2 IRF540, Q3 IRF540, Q4 IRF540, Q5 IRF540, U1 IR2104PBF, U2 IR2104PBF

Commit message: bridge complete. reviewing
Thinking Name
Parts:
- added C5, C6: 100uf, Seeed-Capacitor-2016:PC-D5.3MM
- added D10, D7, D8, D9: (no value), semicon-smd-ipc:MELF-MLL41
- moved R1 5.97 mm to (13.3, 25.8)
- moved R2 4.32 mm to (5.00, 23.5)
- moved R3 4.14 mm to (42.9, 22.9)
- moved OUTPUT 1.00 mm to (30.6, 5.67)
- moved R4 0.95 mm to (30.6, 26.6)
- moved POWER 0.90 mm to (22.0, 5.68)
- moved D1 0.71 mm to (20.6, 39.4)
- moved LOGICINPUT 0.63 mm to (24.8, 47.0)
Connections:
- net GND: now also C5.-, C6.-
- net N$1: now also D8.2
- net N$10: now also D10.1
- net N$3: now also D9.2
- net N$5: now also D10.2
- net N$6: now also D7.2
- net N$7: now also D7.1
- net N$8: now also D8.1
- net N$9: now also D9.1
- net POWER: now also C5.+, C6.+
Routing:
- net POWER: track 155.6 -> 165.4 mm
- net N$8: track 25.0 -> 21.9 mm
- net N$6: track 23.1 -> 20.2 mm
- net N$10: track 15.0 -> 16.8 mm
- net N$5: track 6.49 -> 8.32 mm
- net N$9: track 23.2 -> 21.5 mm
- net N$7: track 47.1 -> 48.7 mm
- net PWM: track 26.3 -> 24.7 mm
- net N$1: track 7.28 -> 8.73 mm
- net IN2: track 18.3 -> 16.9 mm
- net N$3: track 8.49 -> 7.17 mm
- net N$2: track 12.6 -> 13.6 mm
- net VS1: track 74.7 -> 73.8 mm
- net VS2: track 61.7 -> 61.0 mm
- net IN1: track 10.3 -> 9.63 mm
Other:
- board text added: "EjadTech Ejadtech.com"
- board text added: "GND"
- board text added: "OUT1"
- board text added: "OUT2"
- board text added: "VCC"
- board text added: "VCC: 12V-20V"

Commit message: PCB Cosmetics
Parts:
- renumbered LOGICINPUT to INPUT
Other:
- board size 50 x 50 mm -> 49.7 x 49.9 mm
- board text added: "0V"
- board text added: "I1"
- board text added: "I2"
- board text added: "PWM"
Changed lines of the file:
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@@
 <?xml version="1.0" encoding="utf-8"?>
 <!DOCTYPE eagle SYSTEM "eagle.dtd">
-<eagle version="7.6.0">
+<eagle version="7.2.0">
 <drawing>
 <settings>
@@
 <setting verticaltext="up"/>
 </settings>
-<grid distance="0.0125" unitdist="inch" unit="inch" style="lines" multiple="1" display="no" altdistance="0.025" altunitdist="inch" altunit="inch"/>
+<grid distance="0.0125" unitdist="inch" unit="mm" style="lines" multiple="1" display="no" altdistance="0.025" altunitdist="inch" altunit="mm"/>
 <layers>
 <layer number="1" name="Top" color="4" fill="1" visible="yes" active="yes"/>
@@
 <layer number="17" name="Pads" color="2" fill="1" visible="yes" active="yes"/>
 <layer number="18" name="Vias" color="2" fill="1" visible="yes" active="yes"/>
-<layer number="19" name="Unrouted" color="6" fill="1" visible="yes" active="yes"/>
+<layer number="19" name="Unrouted" color="6" fill="1" visible="no" active="yes"/>
 <layer number="20" name="Dimension" color="15" fill="1" visible="yes" active="yes"/>
 <layer number="21" name="tPlace" color="7" fill="1" visible="yes" active="yes"/>
 <layer number="22" name="bPlace" color="7" fill="1" visible="yes" active="yes"/>
-<layer number="23" name="tOrigins" color="15" fill="1" visible="yes" active="yes"/>
-<layer number="24" name="bOrigins" color="15" fill="1" visible="yes" active="yes"/>
+<layer number="23" name="tOrigins" color="15" fill="1" visible="no" active="yes"/>
+<layer number="24" name="bOrigins" color="15" fill="1" visible="no" active="yes"/>
 <layer number="25" name="tNames" color="7" fill="1" visible="yes" active="yes"/>
 <layer number="26" name="bNames" color="7" fill="1" visible="yes" active="yes"/>
@@
 <board>
 <plain>
-<wire x1="0" y1="0" x2="50" y2="0" width="0" layer="20"/>
-<wire x1="50" y1="0" x2="50" y2="50" width="0" layer="20"/>
-<wire x1="50" y1="50" x2="0" y2="50" width="0" layer="20"/>
-<wire x1="0" y1="50" x2="0" y2="0" width="0" layer="20"/>
-<hole x="2.54" y="2.54" drill="2.8"/>
-<hole x="46.99" y="2.54" drill="2.8"/>
-<hole x="46.99" y="46.99" drill="2.8"/>
-<hole x="2.54" y="46.99" drill="2.8"/>
+<wire x1="0.3175" y1="2.2225" x2="2.54" y2="0" width="0" layer="20" curve="90"/>
+<wire x1="2.54" y1="0" x2="46.99" y2="0" width="0" layer="20"/>
+<wire x1="46.99" y1="0" x2="50" y2="2.375" width="0" layer="20" curve="90"/>
+<wire x1="50" y1="2.375" x2="50" y2="43.815" width="0" layer="20"/>
+<wire x1="50" y1="43.815" x2="49.8475" y2="46.3425" width="0" layer="20"/>
+<wire x1="49.8475" y1="46.3425" x2="45.8725" y2="49.8475" width="0" layer="20" curve="90"/>
+<wire x1="45.8725" y1="49.8475" x2="2.3875" y2="49.8475" width="0" layer="20"/>
+<wire x1="2.3875" y1="49.8475" x2="0.3175" y2="47.46" width="0" layer="20" curve="90"/>
+<wire x1="0.3175" y1="47.46" x2="0.3175" y2="2.2225" width="0" layer="20"/>
 <text x="26.035" y="0.635" size="1.016" layer="25" font="vector" ratio="12">OUT1</text>
 <text x="30.7975" y="0.635" size="1.016" layer="25" font="vector" ratio="12">OUT2</text>
@@
 <text x="25.7175" y="26.035" size="1.016" layer="25" font="vector" ratio="12" rot="R90">EjadTech
 Ejadtech.com</text>
+<text x="30.48" y="49.53" size="1.016" layer="25" font="vector" ratio="12" rot="R180">0V</text>
+<text x="21.9075" y="49.53" size="1.016" layer="25" font="vector" ratio="12" rot="R180">I1</text>
+<text x="24.4475" y="49.53" size="1.016" layer="25" font="vector" ratio="12" rot="R180">I2</text>
+<text x="27.94" y="49.53" size="1.016" layer="25" font="vector" ratio="12" rot="R180">PWM</text>
 </plain>
 <attributes>
@@
 <attribute name="VALUE" x="50.419" y="35.433" size="1.27" layer="27" ratio="10" rot="R90"/>
 </element>
-<element name="LOGICINPUT" library="Seeed-Connector -2016" package="H4-2.54" value="4p-2.54" x="24.825" y="47.03" smashed="yes" rot="R90">
+<element name="INPUT" library="Seeed-Connector -2016" package="H4-2.54" value="4p-2.54" x="24.825" y="47.03" smashed="yes" rot="R90">
 <attribute name="MPN" value="F185-1104A1BSYA1" x="24.825" y="47.03" size="1.778" layer="27" rot="R90" display="off"/>
-<attribute name="NAME" x="29.905" y="45.125" size="1.016" layer="25" font="vector" ratio="12" rot="R180"/>
+<attribute name="NAME" x="27.0475" y="45.4425" size="1.016" layer="25" font="vector" ratio="12" rot="R180"/>
 <attribute name="VALUE" x="26.73" y="49.57" size="0.889" layer="27" ratio="11" rot="R180"/>
 </element>
 <element name="OUTPUT" library="Seeed-Connector -2016" package="H2-3.5-7.0X7.0MM" value="GREEN-2P-3.5" x="30.5925" y="5.6675" smashed="yes">
-<attribute name="NAME" x="28.37" y="2.4925" size="1.016" layer="25" font="vector" ratio="12"/>
+<attribute name="NAME" x="35.925" y="2.6525" size="1.016" layer="25" font="vector" ratio="12" rot="R90"/>
 <attribute name="VALUE" x="28.6875" y="1.2225" size="0.889" layer="27" ratio="11"/>
 </element>
 <element name="POWER" library="Seeed-Connector -2016" package="H2-3.5-7.0X7.0MM" value="GREEN-2P-3.5" x="22.02" y="5.685" smashed="yes" rot="R180">
-<attribute name="NAME" x="23.925" y="3.4625" size="1.016" layer="25" font="vector" ratio="12" rot="R180"/>
+<attribute name="NAME" x="25.7475" y="7.7325" size="1.016" layer="25" font="vector" ratio="12" rot="R270"/>
 <attribute name="VALUE" x="23.925" y="10.13" size="0.889" layer="27" ratio="11" rot="R180"/>
 </element>
@@
 <signals>
 <signal name="IN1">
-<contactref element="LOGICINPUT" pad="1"/>
+<contactref element="INPUT" pad="1"/>
 <contactref element="U1" pad="2"/>
 <wire x1="15.3" y1="46.93" x2="15.24" y2="46.99" width="0.4064" layer="16"/>
@@
 </signal>
 <signal name="IN2">
-<contactref element="LOGICINPUT" pad="2"/>
+<contactref element="INPUT" pad="2"/>
 <contactref element="U2" pad="2"/>
 <wire x1="33.22" y1="43.39" x2="33.22" y2="42.745" width="0.3048" layer="16"/>
@@
 </signal>
 <signal name="PWM">
-<contactref element="LOGICINPUT" pad="3"/>
+<contactref element="INPUT" pad="3"/>
 <contactref element="U1" pad="3"/>
 <contactref element="U2" pad="3"/>
@@
 </signal>
 <signal name="GND">
-<contactref element="LOGICINPUT" pad="4"/>
+<contactref element="INPUT" pad="4"/>
 <contactref element="POWER" pad="2"/>
 <contactref element="U2" pad="4"/>
@@
 <wire x1="7.8425" y1="21.91" x2="6.275" y2="23.4775" width="0.3048" layer="16"/>
 </signal>
+<signal name="N$11">
+<via x="2.54" y="46.99" extent="1-16" drill="2.8"/>
+<via x="2.54" y="2.54" extent="1-16" drill="2.8"/>
+<via x="46.99" y="2.54" extent="1-16" drill="2.8"/>
+<via x="46.99" y="46.99" extent="1-16" drill="2.8"/>
+<wire x1="2.54" y1="46.99" x2="46.99" y2="46.99" width="0" layer="19" extent="1-1"/>
+<wire x1="46.99" y1="2.54" x2="46.99" y2="46.99" width="0" layer="19" extent="1-1"/>
+<wire x1="2.54" y1="2.54" x2="2.54" y2="46.99" width="0" layer="19" extent="1-1"/>
+</signal>
 </signals>

Commit message: Revert "PCB Cosmetics"
This reverts commit 40f95e063b70cdd7ef0c66ddfb49b8478f35fe8d.
Parts:
- renumbered INPUT to LOGICINPUT
Other:
- board size 49.7 x 49.9 mm -> 50 x 50 mm
- board text removed: "0V"
- board text removed: "I1"
- board text removed: "I2"
- board text removed: "PWM"
Changed lines of the file:
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@@
 <?xml version="1.0" encoding="utf-8"?>
 <!DOCTYPE eagle SYSTEM "eagle.dtd">
-<eagle version="7.2.0">
+<eagle version="7.6.0">
 <drawing>
 <settings>
@@
 <setting verticaltext="up"/>
 </settings>
-<grid distance="0.0125" unitdist="inch" unit="mm" style="lines" multiple="1" display="no" altdistance="0.025" altunitdist="inch" altunit="mm"/>
+<grid distance="0.0125" unitdist="inch" unit="inch" style="lines" multiple="1" display="no" altdistance="0.025" altunitdist="inch" altunit="inch"/>
 <layers>
 <layer number="1" name="Top" color="4" fill="1" visible="yes" active="yes"/>
@@
 <layer number="17" name="Pads" color="2" fill="1" visible="yes" active="yes"/>
 <layer number="18" name="Vias" color="2" fill="1" visible="yes" active="yes"/>
-<layer number="19" name="Unrouted" color="6" fill="1" visible="no" active="yes"/>
+<layer number="19" name="Unrouted" color="6" fill="1" visible="yes" active="yes"/>
 <layer number="20" name="Dimension" color="15" fill="1" visible="yes" active="yes"/>
 <layer number="21" name="tPlace" color="7" fill="1" visible="yes" active="yes"/>
 <layer number="22" name="bPlace" color="7" fill="1" visible="yes" active="yes"/>
-<layer number="23" name="tOrigins" color="15" fill="1" visible="no" active="yes"/>
-<layer number="24" name="bOrigins" color="15" fill="1" visible="no" active="yes"/>
+<layer number="23" name="tOrigins" color="15" fill="1" visible="yes" active="yes"/>
+<layer number="24" name="bOrigins" color="15" fill="1" visible="yes" active="yes"/>
 <layer number="25" name="tNames" color="7" fill="1" visible="yes" active="yes"/>
 <layer number="26" name="bNames" color="7" fill="1" visible="yes" active="yes"/>
@@
 <board>
 <plain>
-<wire x1="0.3175" y1="2.2225" x2="2.54" y2="0" width="0" layer="20" curve="90"/>
-<wire x1="2.54" y1="0" x2="46.99" y2="0" width="0" layer="20"/>
-<wire x1="46.99" y1="0" x2="50" y2="2.375" width="0" layer="20" curve="90"/>
-<wire x1="50" y1="2.375" x2="50" y2="43.815" width="0" layer="20"/>
-<wire x1="50" y1="43.815" x2="49.8475" y2="46.3425" width="0" layer="20"/>
-<wire x1="49.8475" y1="46.3425" x2="45.8725" y2="49.8475" width="0" layer="20" curve="90"/>
-<wire x1="45.8725" y1="49.8475" x2="2.3875" y2="49.8475" width="0" layer="20"/>
-<wire x1="2.3875" y1="49.8475" x2="0.3175" y2="47.46" width="0" layer="20" curve="90"/>
-<wire x1="0.3175" y1="47.46" x2="0.3175" y2="2.2225" width="0" layer="20"/>
+<wire x1="0" y1="0" x2="50" y2="0" width="0" layer="20"/>
+<wire x1="50" y1="0" x2="50" y2="50" width="0" layer="20"/>
+<wire x1="50" y1="50" x2="0" y2="50" width="0" layer="20"/>
+<wire x1="0" y1="50" x2="0" y2="0" width="0" layer="20"/>
+<hole x="2.54" y="2.54" drill="2.8"/>
+<hole x="46.99" y="2.54" drill="2.8"/>
+<hole x="46.99" y="46.99" drill="2.8"/>
+<hole x="2.54" y="46.99" drill="2.8"/>
 <text x="26.035" y="0.635" size="1.016" layer="25" font="vector" ratio="12">OUT1</text>
 <text x="30.7975" y="0.635" size="1.016" layer="25" font="vector" ratio="12">OUT2</text>
@@
 <text x="25.7175" y="26.035" size="1.016" layer="25" font="vector" ratio="12" rot="R90">EjadTech
 Ejadtech.com</text>
-<text x="30.48" y="49.53" size="1.016" layer="25" font="vector" ratio="12" rot="R180">0V</text>
-<text x="21.9075" y="49.53" size="1.016" layer="25" font="vector" ratio="12" rot="R180">I1</text>
-<text x="24.4475" y="49.53" size="1.016" layer="25" font="vector" ratio="12" rot="R180">I2</text>
-<text x="27.94" y="49.53" size="1.016" layer="25" font="vector" ratio="12" rot="R180">PWM</text>
 </plain>
 <attributes>
@@
 <attribute name="VALUE" x="50.419" y="35.433" size="1.27" layer="27" ratio="10" rot="R90"/>
 </element>
-<element name="INPUT" library="Seeed-Connector -2016" package="H4-2.54" value="4p-2.54" x="24.825" y="47.03" smashed="yes" rot="R90">
+<element name="LOGICINPUT" library="Seeed-Connector -2016" package="H4-2.54" value="4p-2.54" x="24.825" y="47.03" smashed="yes" rot="R90">
 <attribute name="MPN" value="F185-1104A1BSYA1" x="24.825" y="47.03" size="1.778" layer="27" rot="R90" display="off"/>
-<attribute name="NAME" x="27.0475" y="45.4425" size="1.016" layer="25" font="vector" ratio="12" rot="R180"/>
+<attribute name="NAME" x="29.905" y="45.125" size="1.016" layer="25" font="vector" ratio="12" rot="R180"/>
 <attribute name="VALUE" x="26.73" y="49.57" size="0.889" layer="27" ratio="11" rot="R180"/>
 </element>
 <element name="OUTPUT" library="Seeed-Connector -2016" package="H2-3.5-7.0X7.0MM" value="GREEN-2P-3.5" x="30.5925" y="5.6675" smashed="yes">
-<attribute name="NAME" x="35.925" y="2.6525" size="1.016" layer="25" font="vector" ratio="12" rot="R90"/>
+<attribute name="NAME" x="28.37" y="2.4925" size="1.016" layer="25" font="vector" ratio="12"/>
 <attribute name="VALUE" x="28.6875" y="1.2225" size="0.889" layer="27" ratio="11"/>
 </element>
 <element name="POWER" library="Seeed-Connector -2016" package="H2-3.5-7.0X7.0MM" value="GREEN-2P-3.5" x="22.02" y="5.685" smashed="yes" rot="R180">
-<attribute name="NAME" x="25.7475" y="7.7325" size="1.016" layer="25" font="vector" ratio="12" rot="R270"/>
+<attribute name="NAME" x="23.925" y="3.4625" size="1.016" layer="25" font="vector" ratio="12" rot="R180"/>
 <attribute name="VALUE" x="23.925" y="10.13" size="0.889" layer="27" ratio="11" rot="R180"/>
 </element>
@@
 <signals>
 <signal name="IN1">
-<contactref element="INPUT" pad="1"/>
+<contactref element="LOGICINPUT" pad="1"/>
 <contactref element="U1" pad="2"/>
 <wire x1="15.3" y1="46.93" x2="15.24" y2="46.99" width="0.4064" layer="16"/>
@@
 </signal>
 <signal name="IN2">
-<contactref element="INPUT" pad="2"/>
+<contactref element="LOGICINPUT" pad="2"/>
 <contactref element="U2" pad="2"/>
 <wire x1="33.22" y1="43.39" x2="33.22" y2="42.745" width="0.3048" layer="16"/>
@@
 </signal>
 <signal name="PWM">
-<contactref element="INPUT" pad="3"/>
+<contactref element="LOGICINPUT" pad="3"/>
 <contactref element="U1" pad="3"/>
 <contactref element="U2" pad="3"/>
@@
 </signal>
 <signal name="GND">
-<contactref element="INPUT" pad="4"/>
+<contactref element="LOGICINPUT" pad="4"/>
 <contactref element="POWER" pad="2"/>
 <contactref element="U2" pad="4"/>
@@
 <wire x1="7.8425" y1="21.91" x2="6.275" y2="23.4775" width="0.3048" layer="16"/>
 </signal>
-<signal name="N$11">
-<via x="2.54" y="46.99" extent="1-16" drill="2.8"/>
-<via x="2.54" y="2.54" extent="1-16" drill="2.8"/>
-<via x="46.99" y="2.54" extent="1-16" drill="2.8"/>
-<via x="46.99" y="46.99" extent="1-16" drill="2.8"/>
-<wire x1="2.54" y1="46.99" x2="46.99" y2="46.99" width="0" layer="19" extent="1-1"/>
-<wire x1="46.99" y1="2.54" x2="46.99" y2="46.99" width="0" layer="19" extent="1-1"/>
-<wire x1="2.54" y1="2.54" x2="2.54" y2="46.99" width="0" layer="19" extent="1-1"/>
-</signal>
 </signals>

Commit message: silk adjusted
Parts:
- moved C3 39.4 mm to (47.7, 9.53), turned to 180 degrees
- moved D6 36.5 mm to (12.8, 48.3), turned to 180 degrees
- moved D4 36.1 mm to (12.7, 3.38), turned to 180 degrees
- moved C4 35.2 mm to (47.7, 15.2), turned to 180 degrees
- moved C5 35.2 mm to (3.91, 12.7), turned to 270 degrees
- moved D3 32.7 mm to (12.6, 6.32), turned to 0 degrees
- moved D5 32.6 mm to (12.8, 45.1), turned to 0 degrees
- moved C6 31.6 mm to (4.23, 36.2), turned to 270 degrees
- moved D2 29.7 mm to (10.3, 40.6), turned to 180 degrees
- moved OUTPUT 29.5 mm to (45.2, 31.2), turned to 90 degrees
- moved D8 28.8 mm to (30.2, 6.03), turned to 90 degrees
- moved POWER 28.7 mm to (45.2, 22.7), turned to 270 degrees
- moved R2 28.6 mm to (27.3, 5.64), turned to 90 degrees
- moved LOGICINPUT 27.6 mm to (5.14, 27.7), turned to 180 degrees
- moved Q3 27.3 mm to (30.1, 7.10), turned to 270 degrees
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Routing:
- net N$7: track 48.7 -> 25.8 mm, vias 0 -> 1
- net N$6: track 20.2 -> 6.99 mm, vias 1 -> 0
- net POWER: track 165.4 -> 174.1 mm
- net N$4: track 13.5 -> 9.08 mm
- net IN2: track 16.9 -> 13.6 mm
- net VS1: track 73.8 -> 75.8 mm
- net N$2: track 13.6 -> 15.1 mm
- net VS2: track 61.0 -> 59.8 mm
- net PWM: track 24.7 -> 26.0 mm
- net N$5: track 8.32 -> 8.94 mm
Other:
- board size 50 x 50 mm -> 49.9 x 49.9 mm
- board text added: "IN1"
- board text added: "IN2"
- board text added: "NAME"
- board text added: "PWM"

Commit message: final reviewed. Completed
Parts:
- removed LOGICINPUT: 4p-2.54, Seeed-Connector -2016:H4-2.54
- added INPUT: 4p-2.54, Seeed-Connector -2016:H4-2.54
- moved C3 39.7 mm to (8.57, 3.17), turned to 90 degrees
- moved D4 36.2 mm to (2.58, 38.2), turned to 90 degrees
- moved D6 36.2 mm to (47.3, 37.5), turned to 90 degrees
- moved C4 35.5 mm to (14.3, 3.17), turned to 90 degrees
- moved C5 35.2 mm to (11.7, 47.0), turned to 180 degrees
- moved D3 32.8 mm to (5.36, 38.3), turned to 270 degrees
- moved D5 32.2 mm to (44.1, 37.5), turned to 270 degrees
- moved C6 31.3 mm to (33.7, 47.0), turned to 180 degrees
- moved OUTPUT 29.6 mm to (30.3, 5.67), turned to 0 degrees
- moved D2 29.4 mm to (39.7, 40.6), turned to 90 degrees
- moved D8 29.0 mm to (5.08, 20.6), turned to 180 degrees
- moved POWER 29.0 mm to (21.7, 5.68), turned to 180 degrees
- moved R2 28.8 mm to (4.69, 23.5), turned to 180 degrees
- moved Q3 27.6 mm to (6.15, 20.8), turned to 180 degrees
- moved Q4 26.2 mm to (42.5, 20.2), turned to 180 degrees
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Connections:
- net GND: now also INPUT.4; no longer LOGICINPUT.4
- net IN1: now also INPUT.1; no longer LOGICINPUT.1
- net IN2: now also INPUT.2; no longer LOGICINPUT.2
- net PWM: now also INPUT.3; no longer LOGICINPUT.3
Routing:
- net N$7: track 25.8 -> 48.7 mm, vias 1 -> 0
- net N$6: track 6.99 -> 20.2 mm, vias 0 -> 1
- net POWER: track 174.1 -> 165.4 mm
- net N$4: track 9.08 -> 13.5 mm
- net IN2: track 13.6 -> 16.9 mm
- net VS1: track 75.8 -> 73.8 mm
- net N$2: track 15.1 -> 13.6 mm
- net VS2: track 59.8 -> 61.0 mm
- net PWM: track 26.0 -> 24.7 mm
- net N$5: track 8.94 -> 8.32 mm
Other:
- board size 49.9 x 49.9 mm -> 49.8 x 49.8 mm
- board text added: "0V"
- board text added: "I1"
- board text added: "I2"
- board text added: "Logic Voltage: 3V, 5V and 15V"
- board text removed: "IN1"
- board text removed: "IN2"
- board text removed: "NAME"
