File: Schematic_motor_driver.sch (EAGLE design)
At the start: 23 parts, among them Q2 IRF540, Q3 IRF540, Q4 IRF540, Q5 IRF540, U1 IR2104PBF, U2 IR2104PBF

Commit message: bridge complete. reviewing
Thinking Name
Parts:
- added C5, C6: 100uf, Seeed-Capacitor-2016:DIP-ALUMINUM-100UF-16V(D5-H7MM)
- added D10, D7, D8, D9: (no value), semicon-smd-ipc:D-FILL-MLL-41
Connections:
- net GND: now also C5.-, C6.-
- net N$1: now also D8.A
- net N$10: now also D10.C
- net N$3: now also D9.A
- net N$5: now also D10.A
- net N$6: now also D7.A
- net N$7: now also D7.C
- net N$8: now also D8.C
- net N$9: now also D9.C
- net POWER: now also C5.+, C6.+
Changed lines of the file:
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@@
 <setting verticaltext="up"/>
 </settings>
-<grid distance="0.05" unitdist="inch" unit="inch" style="lines" multiple="1" display="yes" altdistance="0.01" altunitdist="inch" altunit="inch"/>
+<grid distance="0.05" unitdist="inch" unit="inch" style="lines" multiple="1" display="no" altdistance="0.01" altunitdist="inch" altunit="inch"/>
 <layers>
 <layer number="1" name="Top" color="4" fill="1" visible="no" active="no"/>
@@
 <part name="C3" library="Seeed-Capacitor-2016" deviceset="DIP-ALUMINUM-100UF-16V(D5-H7MM)" device="" value="100uf"/>
 <part name="C4" library="Seeed-Capacitor-2016" deviceset="DIP-ALUMINUM-100UF-16V(D5-H7MM)" device="" value="100uf"/>
+<part name="D7" library="semicon-smd-ipc" deviceset="D-FILL-" device="MLL-41"/>
+<part name="D8" library="semicon-smd-ipc" deviceset="D-FILL-" device="MLL-41"/>
+<part name="D9" library="semicon-smd-ipc" deviceset="D-FILL-" device="MLL-41"/>
+<part name="D10" library="semicon-smd-ipc" deviceset="D-FILL-" device="MLL-41"/>
+<part name="C5" library="Seeed-Capacitor-2016" deviceset="DIP-ALUMINUM-100UF-16V(D5-H7MM)" device="" value="100uf"/>
+<part name="C6" library="Seeed-Capacitor-2016" deviceset="DIP-ALUMINUM-100UF-16V(D5-H7MM)" device="" value="100uf"/>
 </parts>
 <sheets>
@@
 <instance part="C3" gate="G$1" x="-27.94" y="87.63" rot="R270"/>
 <instance part="C4" gate="G$1" x="-38.1" y="87.63" rot="R270"/>
+<instance part="D7" gate="G$1" x="81.28" y="111.76" rot="R180"/>
+<instance part="D8" gate="G$1" x="86.36" y="68.58" rot="R180"/>
+<instance part="D9" gate="G$1" x="83.82" y="55.88" rot="R180"/>
+<instance part="D10" gate="G$1" x="86.36" y="15.24" rot="R180"/>
+<instance part="C5" gate="G$1" x="-49.53" y="87.63" rot="R270"/>
+<instance part="C6" gate="G$1" x="-59.69" y="87.63" rot="R270"/>
 </instances>
 <busses>
@@
 <wire x1="-38.1" y1="77.47" x2="-38.1" y2="83.82" width="0.1524" layer="91"/>
 <label x="-33.02" y="77.47" size="1.778" layer="95" rot="R270" xref="yes"/>
+<wire x1="-38.1" y1="77.47" x2="-49.53" y2="77.47" width="0.1524" layer="91"/>
+<junction x="-38.1" y="77.47"/>
+<pinref part="C5" gate="G$1" pin="-"/>
+<wire x1="-49.53" y1="77.47" x2="-49.53" y2="83.82" width="0.1524" layer="91"/>
+<pinref part="C6" gate="G$1" pin="-"/>
+<wire x1="-59.69" y1="83.82" x2="-59.69" y2="77.47" width="0.1524" layer="91"/>
+<wire x1="-59.69" y1="77.47" x2="-49.53" y2="77.47" width="0.1524" layer="91"/>
+<junction x="-49.53" y="77.47"/>
 </segment>
 </net>
@@
 <wire x1="-38.1" y1="99.06" x2="-38.1" y2="91.44" width="0.1524" layer="91"/>
 <label x="-33.02" y="99.06" size="1.778" layer="95" rot="R90" xref="yes"/>
+<pinref part="C5" gate="G$1" pin="+"/>
+<wire x1="-49.53" y1="91.44" x2="-49.53" y2="99.06" width="0.1524" layer="91"/>
+<wire x1="-49.53" y1="99.06" x2="-48.26" y2="99.06" width="0.1524" layer="91"/>
+<junction x="-38.1" y="99.06"/>
+<pinref part="C6" gate="G$1" pin="+"/>
+<wire x1="-48.26" y1="99.06" x2="-38.1" y2="99.06" width="0.1524" layer="91"/>
+<wire x1="-59.69" y1="91.44" x2="-59.69" y2="99.06" width="0.1524" layer="91"/>
+<wire x1="-59.69" y1="99.06" x2="-49.53" y2="99.06" width="0.1524" layer="91"/>
 </segment>
 </net>
@@
 <pinref part="R3" gate="G$1" pin="2"/>
 <pinref part="Q4" gate="G$1" pin="G"/>
-<wire x1="88.9" y1="45.72" x2="93.98" y2="45.72" width="0.1524" layer="91"/>
+<wire x1="88.9" y1="45.72" x2="91.44" y2="45.72" width="0.1524" layer="91"/>
+<pinref part="D9" gate="G$1" pin="A"/>
+<wire x1="91.44" y1="45.72" x2="93.98" y2="45.72" width="0.1524" layer="91"/>
+<wire x1="86.36" y1="55.88" x2="91.44" y2="55.88" width="0.1524" layer="91"/>
+<wire x1="91.44" y1="55.88" x2="91.44" y2="45.72" width="0.1524" layer="91"/>
+<junction x="91.44" y="45.72"/>
 </segment>
 </net>
@@
 <pinref part="Q5" gate="G$1" pin="G"/>
 <pinref part="R4" gate="G$1" pin="2"/>
-<wire x1="93.98" y1="24.13" x2="88.9" y2="24.13" width="0.1524" layer="91"/>
+<wire x1="93.98" y1="24.13" x2="91.44" y2="24.13" width="0.1524" layer="91"/>
+<pinref part="D10" gate="G$1" pin="A"/>
+<wire x1="91.44" y1="24.13" x2="88.9" y2="24.13" width="0.1524" layer="91"/>
+<wire x1="88.9" y1="15.24" x2="91.44" y2="15.24" width="0.1524" layer="91"/>
+<wire x1="91.44" y1="15.24" x2="91.44" y2="24.13" width="0.1524" layer="91"/>
+<junction x="91.44" y="24.13"/>
 </segment>
 </net>
@@
 <pinref part="Q2" gate="G$1" pin="G"/>
 <pinref part="R1" gate="G$1" pin="2"/>
-<wire x1="93.98" y1="99.06" x2="88.9" y2="99.06" width="0.1524" layer="91"/>
+<wire x1="93.98" y1="99.06" x2="91.44" y2="99.06" width="0.1524" layer="91"/>
+<pinref part="D7" gate="G$1" pin="A"/>
+<wire x1="91.44" y1="99.06" x2="88.9" y2="99.06" width="0.1524" layer="91"/>
+<wire x1="83.82" y1="111.76" x2="91.44" y2="111.76" width="0.1524" layer="91"/>
+<wire x1="91.44" y1="111.76" x2="91.44" y2="99.06" width="0.1524" layer="91"/>
+<junction x="91.44" y="99.06"/>
 </segment>
 </net>
@@
 <segment>
 <pinref part="R1" gate="G$1" pin="1"/>
-<wire x1="81.28" y1="99.06" x2="72.39" y2="99.06" width="0.1524" layer="91"/>
+<wire x1="81.28" y1="99.06" x2="76.2" y2="99.06" width="0.1524" layer="91"/>
+<wire x1="76.2" y1="99.06" x2="72.39" y2="99.06" width="0.1524" layer="91"/>
 <wire x1="72.39" y1="99.06" x2="72.39" y2="96.52" width="0.1524" layer="91"/>
 <pinref part="U1" gate="A" pin="HO"/>
 <wire x1="72.39" y1="96.52" x2="71.12" y2="96.52" width="0.1524" layer="91"/>
+<pinref part="D7" gate="G$1" pin="C"/>
+<wire x1="78.74" y1="111.76" x2="76.2" y2="111.76" width="0.1524" layer="91"/>
+<wire x1="76.2" y1="111.76" x2="76.2" y2="99.06" width="0.1524" layer="91"/>
+<junction x="76.2" y="99.06"/>
 </segment>
 </net>
@@
 <wire x1="72.39" y1="93.98" x2="72.39" y2="78.74" width="0.1524" layer="91"/>
 <pinref part="R2" gate="G$1" pin="1"/>
-<wire x1="72.39" y1="78.74" x2="81.28" y2="78.74" width="0.1524" layer="91"/>
+<wire x1="72.39" y1="78.74" x2="76.2" y2="78.74" width="0.1524" layer="91"/>
+<pinref part="D8" gate="G$1" pin="C"/>
+<wire x1="76.2" y1="78.74" x2="81.28" y2="78.74" width="0.1524" layer="91"/>
+<wire x1="83.82" y1="68.58" x2="76.2" y2="68.58" width="0.1524" layer="91"/>
+<wire x1="76.2" y1="68.58" x2="76.2" y2="78.74" width="0.1524" layer="91"/>
+<junction x="76.2" y="78.74"/>
 </segment>
 </net>
@@
 <pinref part="R3" gate="G$1" pin="1"/>
 <wire x1="77.47" y1="45.72" x2="81.28" y2="45.72" width="0.1524" layer="91"/>
+<pinref part="D9" gate="G$1" pin="C"/>
+<wire x1="81.28" y1="55.88" x2="77.47" y2="55.88" width="0.1524" layer="91"/>
+<wire x1="77.47" y1="55.88" x2="77.47" y2="46.99" width="0.1524" layer="91"/>
+<junction x="77.47" y="46.99"/>
 </segment>
 </net>
@@
 <pinref part="R4" gate="G$1" pin="1"/>
 <wire x1="77.47" y1="24.13" x2="81.28" y2="24.13" width="0.1524" layer="91"/>
+<pinref part="D10" gate="G$1" pin="C"/>
+<wire x1="83.82" y1="15.24" x2="77.47" y2="15.24" width="0.1524" layer="91"/>
+<wire x1="77.47" y1="15.24" x2="77.47" y2="24.13" width="0.1524" layer="91"/>
+<junction x="77.47" y="24.13"/>
 </segment>
 </net>
@@
 <pinref part="R2" gate="G$1" pin="2"/>
 <pinref part="Q3" gate="G$1" pin="G"/>
-<wire x1="88.9" y1="78.74" x2="93.98" y2="78.74" width="0.1524" layer="91"/>
-</segment>
-</net>
+<wire x1="88.9" y1="78.74" x2="90.17" y2="78.74" width="0.1524" layer="91"/>
+<pinref part="D8" gate="G$1" pin="A"/>
+<wire x1="90.17" y1="78.74" x2="93.98" y2="78.74" width="0.1524" layer="91"/>
+<wire x1="88.9" y1="68.58" x2="90.17" y2="68.58" width="0.1524" layer="91"/>
+<wire x1="90.17" y1="68.58" x2="90.17" y2="78.74" width="0.1524" layer="91"/>
+<junction x="90.17" y="78.74"/>
+</segment>
+</net>

Commit message: final reviewed. Completed
Parts:
- renumbered LOGICINPUT to INPUT
Changed lines of the file:
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@@
 <?xml version="1.0" encoding="utf-8"?>
 <!DOCTYPE eagle SYSTEM "eagle.dtd">
-<eagle version="7.6.0">
+<eagle version="7.2.0">
 <drawing>
 <settings>
@@
 <setting verticaltext="up"/>
 </settings>
-<grid distance="0.05" unitdist="inch" unit="inch" style="lines" multiple="1" display="no" altdistance="0.01" altunitdist="inch" altunit="inch"/>
+<grid distance="0.1" unitdist="inch" unit="inch" style="lines" multiple="1" display="no" altdistance="0.01" altunitdist="inch" altunit="inch"/>
 <layers>
 <layer number="1" name="Top" color="4" fill="1" visible="no" active="no"/>
@@
 <part name="U1" library="International_Rectifier_By_element14_Batch_1" deviceset="IR2104PBF" device=""/>
 <part name="U2" library="International_Rectifier_By_element14_Batch_1" deviceset="IR2104PBF" device=""/>
-<part name="LOGICINPUT" library="Seeed-Connector -2016" deviceset="DIP-BLACK-FEMALE-HEADER-VERT(4P-2.54)" device="" value="4p-2.54"/>
+<part name="INPUT" library="Seeed-Connector -2016" deviceset="DIP-BLACK-FEMALE-HEADER-VERT(4P-2.54)" device="" value="4p-2.54"/>
 <part name="POWER" library="Seeed-Connector -2016" deviceset="SCREW-TERMINAL-GREEN(2P-3.5)" device="" value="GREEN-2P-3.5"/>
 <part name="D1" library="adafruit" deviceset="1N4004" device=""/>
@@
 <instance part="U1" gate="A" x="53.34" y="88.9"/>
 <instance part="U2" gate="A" x="53.34" y="39.37"/>
-<instance part="LOGICINPUT" gate="G$1" x="1.27" y="66.04"/>
+<instance part="INPUT" gate="G$1" x="1.27" y="66.04"/>
 <instance part="POWER" gate="G$1" x="1.27" y="87.63"/>
 <instance part="D1" gate="1" x="22.86" y="95.25" rot="R270"/>
@@
 <net name="IN1" class="0">
 <segment>
-<pinref part="LOGICINPUT" gate="G$1" pin="P$1"/>
+<pinref part="INPUT" gate="G$1" pin="P$1"/>
 <wire x1="-6.35" y1="69.85" x2="-11.43" y2="69.85" width="0.1524" layer="91"/>
 <label x="-11.43" y="69.85" size="1.778" layer="95" rot="R180" xref="yes"/>
@@
 <net name="IN2" class="0">
 <segment>
-<pinref part="LOGICINPUT" gate="G$1" pin="P$2"/>
+<pinref part="INPUT" gate="G$1" pin="P$2"/>
 <wire x1="-6.35" y1="67.31" x2="-11.43" y2="67.31" width="0.1524" layer="91"/>
 <label x="-11.43" y="67.31" size="1.778" layer="95" rot="R180" xref="yes"/>
@@
 <net name="PWM" class="0">
 <segment>
-<pinref part="LOGICINPUT" gate="G$1" pin="P$3"/>
+<pinref part="INPUT" gate="G$1" pin="P$3"/>
 <wire x1="-11.43" y1="64.77" x2="-6.35" y2="64.77" width="0.1524" layer="91"/>
 <label x="-11.43" y="64.77" size="1.778" layer="95" rot="R180" xref="yes"/>
@@
 <net name="GND" class="0">
 <segment>
-<pinref part="LOGICINPUT" gate="G$1" pin="P$4"/>
+<pinref part="INPUT" gate="G$1" pin="P$4"/>
 <wire x1="-6.35" y1="62.23" x2="-11.43" y2="62.23" width="0.1524" layer="91"/>
 <label x="-11.43" y="62.23" size="1.778" layer="95" rot="R180" xref="yes"/>

Commit message: Revert "PCB Cosmetics"
This reverts commit 40f95e063b70cdd7ef0c66ddfb49b8478f35fe8d.
Parts:
- renumbered INPUT to LOGICINPUT
Changed lines of the file:
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@@
 <?xml version="1.0" encoding="utf-8"?>
 <!DOCTYPE eagle SYSTEM "eagle.dtd">
-<eagle version="7.2.0">
+<eagle version="7.6.0">
 <drawing>
 <settings>
@@
 <setting verticaltext="up"/>
 </settings>
-<grid distance="0.1" unitdist="inch" unit="inch" style="lines" multiple="1" display="no" altdistance="0.01" altunitdist="inch" altunit="inch"/>
+<grid distance="0.05" unitdist="inch" unit="inch" style="lines" multiple="1" display="no" altdistance="0.01" altunitdist="inch" altunit="inch"/>
 <layers>
 <layer number="1" name="Top" color="4" fill="1" visible="no" active="no"/>
@@
 <part name="U1" library="International_Rectifier_By_element14_Batch_1" deviceset="IR2104PBF" device=""/>
 <part name="U2" library="International_Rectifier_By_element14_Batch_1" deviceset="IR2104PBF" device=""/>
-<part name="INPUT" library="Seeed-Connector -2016" deviceset="DIP-BLACK-FEMALE-HEADER-VERT(4P-2.54)" device="" value="4p-2.54"/>
+<part name="LOGICINPUT" library="Seeed-Connector -2016" deviceset="DIP-BLACK-FEMALE-HEADER-VERT(4P-2.54)" device="" value="4p-2.54"/>
 <part name="POWER" library="Seeed-Connector -2016" deviceset="SCREW-TERMINAL-GREEN(2P-3.5)" device="" value="GREEN-2P-3.5"/>
 <part name="D1" library="adafruit" deviceset="1N4004" device=""/>
@@
 <instance part="U1" gate="A" x="53.34" y="88.9"/>
 <instance part="U2" gate="A" x="53.34" y="39.37"/>
-<instance part="INPUT" gate="G$1" x="1.27" y="66.04"/>
+<instance part="LOGICINPUT" gate="G$1" x="1.27" y="66.04"/>
 <instance part="POWER" gate="G$1" x="1.27" y="87.63"/>
 <instance part="D1" gate="1" x="22.86" y="95.25" rot="R270"/>
@@
 <net name="IN1" class="0">
 <segment>
-<pinref part="INPUT" gate="G$1" pin="P$1"/>
+<pinref part="LOGICINPUT" gate="G$1" pin="P$1"/>
 <wire x1="-6.35" y1="69.85" x2="-11.43" y2="69.85" width="0.1524" layer="91"/>
 <label x="-11.43" y="69.85" size="1.778" layer="95" rot="R180" xref="yes"/>
@@
 <net name="IN2" class="0">
 <segment>
-<pinref part="INPUT" gate="G$1" pin="P$2"/>
+<pinref part="LOGICINPUT" gate="G$1" pin="P$2"/>
 <wire x1="-6.35" y1="67.31" x2="-11.43" y2="67.31" width="0.1524" layer="91"/>
 <label x="-11.43" y="67.31" size="1.778" layer="95" rot="R180" xref="yes"/>
@@
 <net name="PWM" class="0">
 <segment>
-<pinref part="INPUT" gate="G$1" pin="P$3"/>
+<pinref part="LOGICINPUT" gate="G$1" pin="P$3"/>
 <wire x1="-11.43" y1="64.77" x2="-6.35" y2="64.77" width="0.1524" layer="91"/>
 <label x="-11.43" y="64.77" size="1.778" layer="95" rot="R180" xref="yes"/>
@@
 <net name="GND" class="0">
 <segment>
-<pinref part="INPUT" gate="G$1" pin="P$4"/>
+<pinref part="LOGICINPUT" gate="G$1" pin="P$4"/>
 <wire x1="-6.35" y1="62.23" x2="-11.43" y2="62.23" width="0.1524" layer="91"/>
 <label x="-11.43" y="62.23" size="1.778" layer="95" rot="R180" xref="yes"/>
